File: Power Supply E5/Power Supply E5.kicad_pcb (KiCad board)
At the start: 2 copper layers, 36 parts, among them J1 Conn_01x04, J2 Conn_01x05, J3 Conn_01x06, Q1 TL2575-05IKV, Q2 TL2575-05IKV, U1 LM2592

Commit message: Final changes were made before printing as pdf
Parts:
- removed the Q1 at (0.25, 0.25) (x2)
- removed the Q2 at (0.25, 1.75) (x2)
- removed U1: LM2592, components:TO170P470X1028X2142-5P
- added IC**: TO170P470X1028X2142-5P, Components:TO170P470X1028X2142-5P - Copy, F.Cu at (43.2, 83.8)
- added IC**: TO170P470X1028X2142-5P, Components:TO170P470X1028X2142-5P - Copy, F.Cu at (42.5, 61.8)
- added Q**: TO170P470X1016X2338-5P, Components:TO170P470X1016X2338-5P, F.Cu at (66.0, 20.3)
- D1, D2, D3, D4: value 1N4007 -> 1N5059
- moved D4 5.71 mm to (45.1, 40.6)
- moved LB1 3.64 mm to (78.7, 22.9), turned to -90 degrees
- moved R2 3.25 mm to (48.9, 34.9)
- moved D2 2.54 mm to (40.6, 50.8)
- moved REF** 0.90 mm to (85.7, 111.1)
- moved REF** 0.90 mm to (85.7, 21.0)
- moved REF** 0.90 mm to (21.0, 111.1)
- moved REF** 0.90 mm to (21.0, 21.0)
Routing:
- net /pot2: track 0.00 -> 114.3 mm
- net /pot2w: track 0.00 -> 93.9 mm
- net /5/A COM: track 78.8 -> 169.8 mm
- net /pot2_l: track 0.00 -> 79.7 mm
- net /pot1: track 11.0 -> 65.6 mm
- net /pot1w: track 0.00 -> 44.0 mm
- net Net-(D10-K): track 0.00 -> 35.1 mm
- net /pot1_l: track 0.00 -> 34.4 mm
- net /5V: track 35.8 -> 64.3 mm
- net /-Ch B: track 114.7 -> 141.7 mm
- net Net-(D1-K): track 56.6 -> 74.6 mm
- net Net-(D6-K): track 27.5 -> 42.7 mm
- net /b+: track 7.07 -> 20.7 mm
- net /a-: track 33.7 -> 28.0 mm
- net /Ch B: track 89.0 -> 86.2 mm
Other:
- board outline added: 76.2 x 101.6 mm
- board text added: "Nikolai Stanovich"
