File: Power Supply E5/Power Supply E5.kicad_sch (KiCad schematic)
At the start: 31 parts, among them J1 Conn_01x04, J2 Conn_01x05, J3 Conn_01x06, Q1 TL2575-05IKV, Q2 TL2575-05IKV, T1 Transformer_1P_2S, U1 LM2592

Commit message: Final changes were made before printing as pdf
Parts:
- D1, D2, D3, D4: value 1N4007 -> 1N5059
- Q1, Q2: footprint TO170P470X1016X2338-5P -> Components:TO170P470X1016X2338-5P
- U1: footprint TO170P470X1028X2142-5P -> Components:TO170P470X1028X2142-5P
Connections:
- net 5/A COM: no longer U1.2 (OUTPUT)
- net at D10.1 (K), L5v1.2: now also U1.2 (OUTPUT); no longer U1.5 (~{ON}/OFF)
Other:
- moved on the sheet: L5v1, U1
